File: BMS/BMS.kicad_pcb (KiCad board)
At the start: 2 copper layers, 34 parts, among them U1 ATmega406-1AA

Commit message: DCDC fix unavailable parts, BMS redesign, handle fix, rearrange top half
Parts:
- removed D4: 1N6857, Diode_THT:D_DO-35_SOD27_P7.62mm_Horizontal
- added C1: 1 u, Capacitor_SMD:C_0805_2012Metric, B.Cu at (48.6, 37.8)
- added CRESET1: 0.1 u, Capacitor_SMD:C_0603_1608Metric, F.Cu at (57.4, 39.3)
- added CReg1: 0.1 u, Capacitor_SMD:C_0603_1608Metric, F.Cu at (59.9, 43.7)
- added CReg2: 1 u, Capacitor_SMD:C_0805_2012Metric, F.Cu at (60.0, 41.9)
- added D5: CDBQR0130L-HF, Diode_SMD:D_0402_1005Metric, F.Cu at (74.6, 42.2)
- added H1: MountingHole, MountingHole:MountingHole_2.2mm_M2, F.Cu at (274.6, 45.3)
- added H2: MountingHole, MountingHole:MountingHole_2.2mm_M2, F.Cu at (90.6, 45.4)
- added H3: MountingHole, MountingHole:MountingHole_2.2mm_M2, F.Cu at (20.7, 33.2)
- added H4: MountingHole, MountingHole:MountingHole_2.2mm_M2, F.Cu at (154.1, 33.0)
- added JTag0: Conn_01x04_Pin, Connector_PinHeader_2.00mm:PinHeader_1x04_P2.00mm_Horizontal, F.Cu at (111.8, 39.9)
- added LED0: LED, Diode_SMD:D_0603_1608Metric, F.Cu at (96.2, 38.1)
- added LED1: LED, Diode_SMD:D_0603_1608Metric, F.Cu at (101.4, 38.1)
- added LED2: LED, Diode_SMD:D_0603_1608Metric, F.Cu at (107.4, 38.1)
- added LED3: LED, Diode_SMD:D_0603_1608Metric, F.Cu at (127.3, 38.1)
- added LED4: LED, Diode_SMD:D_0603_1608Metric, F.Cu at (131.6, 38.1)
- added Q1: TPCA8120,L1Q, Library:TPH4R003NLL1Q, F.Cu at (262.0, 38.5)
- added Q2: TPCA8120,L1Q, Library:TPH4R003NLL1Q, F.Cu at (271.1, 38.5)
- added Q3: TPCA8120,L1Q, Library:TPH4R003NLL1Q, F.Cu at (250.2, 38.4)
- added R1: 10 k, Resistor_SMD:R_0402_1005Metric, B.Cu at (50.2, 37.9)
- added RLED-0: 20, Resistor_SMD:R_0402_1005Metric, F.Cu at (96.2, 41.2)
- added RLED-1: 20, Resistor_SMD:R_0402_1005Metric, F.Cu at (101.4, 41.2)
- added RLED-2: 20, Resistor_SMD:R_0402_1005Metric, F.Cu at (107.2, 41.1)
- added RLED-3: 20, Resistor_SMD:R_0402_1005Metric, F.Cu at (127.3, 40.9)
- added RLED-4: 20, Resistor_SMD:R_0402_1005Metric, F.Cu at (131.6, 40.6)
- added RPU1: 2.2 M, Resistor_SMD:R_2010_5025Metric, F.Cu at (77.9, 40.2)
- added RPU2: 2.2 M, Resistor_SMD:R_2010_5025Metric, F.Cu at (68.9, 40.5)
- added RSense0: 5 m, Library:Y14880R00500B9R, F.Cu at (30.5, 40.9)
- added Rcf1: 1 M, Resistor_SMD:R_0402_1005Metric, F.Cu at (258.7, 42.6)
- added Rdf1: 1 M, Resistor_SMD:R_0402_1005Metric, F.Cu at (274.2, 34.5)
- added Rni1: 100, Resistor_SMD:R_0603_1608Metric, F.Cu at (38.9, 44.2)
- added Rpf1: 1 M, Resistor_SMD:R_0402_1005Metric, F.Cu at (256.1, 34.2)
- added Rpi1: 100, Resistor_SMD:R_0603_1608Metric, F.Cu at (38.9, 38.3)
- D3: value 1N6857 -> CDBQR0130L-HF; footprint Diode_THT:D_DO-35_SOD27_P7.62mm_Horizontal -> Diode_SMD:D_0402_1005Metric
- RP0, RP1, RP2, RP3, RP4: value 1 k -> 500; footprint Resistor_SMD:R_0402_1005Metric -> Resistor_SMD:R_1206_3216Metric
- moved B4 303.7 mm to (274.5, 32.6), turned to -90 degrees
- moved RP4 283.8 mm to (268.4, 32.6), turned to -90 degrees
- moved VOut2 281.8 mm to (256.1, 36.6), turned to 180 degrees
- moved D1 280.5 mm to (259.9, 32.6), turned to -90 degrees
- moved RN1 278.0 mm to (263.5, 31.8), turned to -90 degrees
- moved Rpc1 274.4 mm to (258.1, 45.2)
- moved D2 270.8 mm to (254.4, 32.2), turned to -90 degrees
- moved B3 241.8 mm to (212.4, 31.4), turned to -90 degrees
- moved TH4 224.7 mm to (215.5, 46.8), turned to 180 degrees
- moved RP3 224.2 mm to (208.6, 31.3)
- moved B2 183.0 mm to (147.5, 31.4), turned to -90 degrees
- moved TH3 159.9 mm to (150.7, 46.4), turned to 180 degrees
- moved RP2 159.7 mm to (143.6, 31.6)
- moved B1 119.1 mm to (82.2, 31.4), turned to -90 degrees
- moved D3 109.0 mm to (71.8, 42.3), turned to 90 degrees
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Connections:
- D3 pad 1: /SMBUS/SDA -> /SMBUS/SCL
- U1 pad 13: /XTAL/RESET -> Net-(U1-~{RESET})
- U1 pad 14: /XTAL/XTAL1 -> unconnected-(U1-XTAL1-Pad14)
- U1 pad 15: /XTAL/XTAL2 -> unconnected-(U1-XTAL2-Pad15)
Routing:
- net /Battery/PV4: track 0.00 -> 236.3 mm, vias 0 -> 4
- net /FETs/OD: track 0.00 -> 235.2 mm, vias 0 -> 2
- net /FETs/OC: track 0.00 -> 221.3 mm, vias 0 -> 2
- net /Battery/PVT: track 0.00 -> 219.3 mm, vias 0 -> 2
- net /FETs/VFET: track 0.00 -> 219.3 mm, vias 0 -> 2
- net /FETs/OPC: track 0.00 -> 214.9 mm, vias 0 -> 2
- net /FETs/BATT: track 0.00 -> 212.2 mm, vias 0 -> 2
- net /Thermal/PA0: track 0.00 -> 190.6 mm, vias 0 -> 1
- net /Battery/PV3: track 0.00 -> 175.2 mm
- net /Thermal/PA4: track 0.00 -> 168.2 mm
- net GND: track 0.00 -> 161.2 mm, vias 0 -> 20
- net /Battery/PV2: track 0.00 -> 110.8 mm
- net /Thermal/PA3: track 0.00 -> 105.4 mm
- net /LEDs/VREG: track 0.00 -> 90.8 mm, vias 0 -> 2
- net /LEDs/PB4: track 0.00 -> 79.7 mm
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- added copper zone on F.Cu, net /Battery/B0
- added copper zone on F.Cu, net /Battery/B4
- added copper zone on F.Cu, net /FETs/Vout
- added copper zone on B.Cu, net GND
- added copper zone on F.Cu, net GND
- added copper zone on F.Cu, net Net-(Q1-D_1)
- added copper zone on F.Cu, net Net-(Q3-D_1)
Other:
- board outline added: 260 x 18 mm
