File: BMS/fets.kicad_sch (KiCad schematic)
At the start: 9 parts, among them Q1 TPCA8120,L1Q, Q2 TPCA8120,L1Q, Q3 TPCA8120,L1Q

Commit message: DCDC fix unavailable parts, BMS redesign, handle fix, rearrange top half
Parts:
- D1: Manufacturer_Part_Number (none) -> BAV70,215
- D2: Manufacturer_Part_Number (none) -> BAS516,135
- Rcf1, Rdf1, Rpf1: footprint (none) -> Resistor_SMD:R_0402_1005Metric; Manufacturer_Part_Number (none) -> 560112110033
- Rpc1: Manufacturer_Part_Number (none) -> 71-PTN0402Y5000BST1
Connections:
- net Vout: now also Q1.1 (S_1), Q1.2 (S_2), Q1.3 (S_3), Rcf1.2
Changed lines of the file:
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@@
+	)
+	(junction
+		(at 115.57 92.71)
+		(diameter 0)
+		(color 0 0 0 0)
 	)
 	(junction
@@
 	(wire
 		(pts
+			(xy 154.94 87.63) (xy 115.57 87.63)
+		)
+		(stroke
+			(width 0)
+			(type default)
+		)
+	)
+	(wire
+		(pts
 			(xy 72.39 64.77) (xy 102.87 64.77)
 		)
@@
 		(pts
 			(xy 140.97 64.77) (xy 140.97 62.23)
+		)
+		(stroke
+			(width 0)
+			(type default)
+		)
+	)
+	(wire
+		(pts
+			(xy 115.57 87.63) (xy 115.57 92.71)
 		)
 		(stroke
@@
 			)
 		)
-		(property "Footprint" ""
+		(property "Footprint" "Resistor_SMD:R_0402_1005Metric"
 			(at 106.68 61.468 90)
 			(effects
@@
 			)
 		)
-		(property "Datasheet" ""
+		(property "Datasheet" "https://www.we-online.com/components/products/datasheet/560112110033.pdf"
 			(at 106.68 59.69 0)
 			(effects
@@
 		)
 		(property "Description" ""
+			(at 106.68 59.69 0)
+			(effects
+				(font
+					(size 1.27 1.27)
+				)
+				(hide yes)
+			)
+		)
+		(property "Manufacturer_Part_Number" "560112110033"
 			(at 106.68 59.69 0)
 			(effects
@@
 			)
 		)
-		(property "Footprint" ""
+		(property "Footprint" "Resistor_SMD:R_0402_1005Metric"
 			(at 104.14 119.888 90)
 			(effects
@@
 			)
 		)
-		(property "Datasheet" ""
+		(property "Datasheet" "https://www.we-online.com/components/products/datasheet/560112110033.pdf"
 			(at 104.14 118.11 0)
 			(effects
@@
 		)
 		(property "Description" "RCV12061M00FKEAAT"
+			(at 104.14 118.11 0)
+			(effects
+				(font
+					(size 1.27 1.27)
+				)
+				(hide yes)
+			)
+		)
+		(property "Manufacturer_Part_Number" "560112110033 "
 			(at 104.14 118.11 0)
 			(effects
@@
 			)
 		)
-		(property "Footprint" ""
+		(property "Footprint" "Resistor_SMD:R_0402_1005Metric"
 			(at 101.6 97.028 90)
 			(effects
@@
 			)
 		)
-		(property "Datasheet" ""
+		(property "Datasheet" "https://www.we-online.com/components/products/datasheet/560112110033.pdf"
 			(at 101.6 95.25 0)
 			(effects
@@
 		)
 		(property "Description" ""
+			(at 101.6 95.25 0)
+			(effects
+				(font
+					(size 1.27 1.27)
+				)
+				(hide yes)
+			)
+		)
+		(property "Manufacturer_Part_Number" "560112110033"
 			(at 101.6 95.25 0)
 			(effects
@@
 			)
 		)
+		(property "Manufacturer_Part_Number" "71-PTN0402Y5000BST1"
+			(at 140.97 81.28 0)
+			(effects
+				(font
+					(size 1.27 1.27)
+				)
+				(hide yes)
+			)
+		)
 		(pin "1"
 		)
@@
 			)
 		)
+		(property "Manufacturer_Part_Number" "BAS516,135"
+			(at 165.1 106.68 0)
+			(effects
+				(font
+					(size 1.27 1.27)
+				)
+				(hide yes)
+			)
+		)
 		(pin "1"
 		)
@@
 			(at 130.81 144.78 0)
 			(effects
+				(font
+					(size 1.27 1.27)
+				)
+				(hide yes)
+			)
+		)
+		(property "Manufacturer_Part_Number" "BAV70,215"
+			(at 130.81 144.78 0)
+			(effects
