File: BMS/leds.kicad_sch (KiCad schematic)
At the start: 12 parts

Commit message: DCDC fix unavailable parts, BMS redesign, handle fix, rearrange top half
Parts:
- CReg1: footprint (none) -> Capacitor_SMD:C_0603_1608Metric; Manufacturer_Part_Number (none) -> KAM15AR71H104KT
- CReg2: footprint (none) -> Capacitor_SMD:C_0805_2012Metric; Manufacturer_Part_Number (none) -> KGM21AR71H105JU
- LED0, LED1, LED2, LED3, LED4: footprint (none) -> Diode_SMD:D_0603_1608Metric; Manufacturer_Part_Number (none) -> ASCKCA00-BU4V4020502
- RLED-0, RLED-1, RLED-2, RLED-3, RLED-4: footprint (none) -> Resistor_SMD:R_0402_1005Metric; Manufacturer_Part_Number (none) -> ESR01MZPF20R0
Changed lines of the file:
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@@
 			)
 		)
-		(property "Footprint" ""
+		(property "Footprint" "Resistor_SMD:R_0402_1005Metric"
 			(at 50.8 71.628 90)
 			(effects
@@
 			)
 		)
-		(property "Datasheet" "~"
+		(property "Datasheet" "https://hu.mouser.com/datasheet/2/348/esr_e-3009601.pdf"
 			(at 50.8 69.85 0)
 			(effects
@@
 			)
 		)
+		(property "Manufacturer_Part_Number" "ESR01MZPF20R0"
+			(at 50.8 69.85 0)
+			(effects
+				(font
+					(size 1.27 1.27)
+				)
+				(hide yes)
+			)
+		)
 		(pin "2"
 		)
@@
 			)
 		)
-		(property "Footprint" ""
+		(property "Footprint" "Diode_SMD:D_0603_1608Metric"
 			(at 63.5 59.69 0)
 			(effects
@@
 			)
 		)
-		(property "Datasheet" "~"
+		(property "Datasheet" "https://hu.mouser.com/datasheet/2/678/ASCKCx00_xxxxx0x0x02_DS101-3169121.pdf"
 			(at 63.5 59.69 0)
 			(effects
@@
 			)
 		)
+		(property "Manufacturer_Part_Number" "ASCKCA00-BU4V4020502"
+			(at 63.5 59.69 0)
+			(effects
+				(font
+					(size 1.27 1.27)
+				)
+				(hide yes)
+			)
+		)
 		(pin "1"
 		)
@@
 			)
 		)
-		(property "Footprint" ""
+		(property "Footprint" "Resistor_SMD:R_0402_1005Metric"
 			(at 50.8 38.608 90)
 			(effects
@@
 			)
 		)
-		(property "Datasheet" "~"
+		(property "Datasheet" "https://hu.mouser.com/datasheet/2/348/esr_e-3009601.pdf"
 			(at 50.8 36.83 0)
 			(effects
@@
 			)
 		)
+		(property "Manufacturer_Part_Number" "ESR01MZPF20R0"
+			(at 50.8 36.83 0)
+			(effects
+				(font
+					(size 1.27 1.27)
+				)
+				(hide yes)
+			)
+		)
 		(pin "2"
 		)
@@
 			)
 		)
-		(property "Footprint" ""
+		(property "Footprint" "Resistor_SMD:R_0402_1005Metric"
 			(at 50.8 61.468 90)
 			(effects
@@
 			)
 		)
-		(property "Datasheet" "~"
+		(property "Datasheet" "https://hu.mouser.com/datasheet/2/348/esr_e-3009601.pdf"
 			(at 50.8 59.69 0)
 			(effects
@@
 			)
 		)
+		(property "Manufacturer_Part_Number" "ESR01MZPF20R0"
+			(at 50.8 59.69 0)
+			(effects
+				(font
+					(size 1.27 1.27)
+				)
+				(hide yes)
+			)
+		)
 		(pin "2"
 		)
@@
 			)
 		)
-		(property "Footprint" ""
+		(property "Footprint" "Resistor_SMD:R_0402_1005Metric"
 			(at 50.8 83.058 90)
 			(effects
@@
 			)
 		)
-		(property "Datasheet" "~"
+		(property "Datasheet" "https://hu.mouser.com/datasheet/2/348/esr_e-3009601.pdf"
 			(at 50.8 81.28 0)
 			(effects
@@
 			)
 		)
+		(property "Manufacturer_Part_Number" "ESR01MZPF20R0"
+			(at 50.8 81.28 0)
+			(effects
+				(font
+					(size 1.27 1.27)
+				)
+				(hide yes)
+			)
+		)
 		(pin "2"
 		)
@@
 			)
 		)
-		(property "Footprint" ""
+		(property "Footprint" "Diode_SMD:D_0603_1608Metric"
 			(at 63.5 36.83 0)
 			(effects
@@
 			)
 		)
-		(property "Datasheet" "~"
+		(property "Datasheet" "https://hu.mouser.com/datasheet/2/678/ASCKCx00_xxxxx0x0x02_DS101-3169121.pdf"
 			(at 63.5 36.83 0)
 			(effects
@@
 			)
 		)
+		(property "Manufacturer_Part_Number" "ASCKCA00-BU4V4020502"
+			(at 63.5 36.83 0)
+			(effects
+				(font
+					(size 1.27 1.27)
+				)
+				(hide yes)
+			)
+		)
 		(pin "1"
 		)
@@
 			)
 		)
-		(property "Footprint" ""
+		(property "Footprint" "Capacitor_SMD:C_0603_1608Metric"
 			(at 49.2252 106.68 0)
 			(effects
@@
 			)
 		)
-		(property "Datasheet" "~"
+		(property "Datasheet" "https://hu.mouser.com/datasheet/2/40/AutoMLCCKAM-3216307.pdf"
 			(at 48.26 102.87 0)
 			(effects
@@
 			)
 		)
+		(property "Manufacturer_Part_Number" "KAM15AR71H104KT"
+			(at 48.26 102.87 0)
+			(effects
+				(font
+					(size 1.27 1.27)
+				)
+				(hide yes)
+			)
+		)
 		(pin "1"
 		)
@@
 			)
 		)
-		(property "Footprint" ""
+		(property "Footprint" "Capacitor_SMD:C_0805_2012Metric"
 			(at 60.6552 106.68 0)
 			(effects
@@
 			)
 		)
-		(property "Datasheet" "~"
+		(property "Datasheet" "https://hu.mouser.com/datasheet/2/40/KGM_X7R-3223212.pdf"
 			(at 59.69 102.87 0)
 			(effects
@@
 			)
 		)
+		(property "Manufacturer_Part_Number" "KGM21AR71H105JU"
+			(at 59.69 102.87 0)
+			(effects
+				(font
+					(size 1.27 1.27)
+				)
+				(hide yes)
+			)
+		)
 		(pin "1"
 		)
@@
 			)
 		)
-		(property "Footprint" ""
+		(property "Footprint" "Resistor_SMD:R_0402_1005Metric"
 			(at 50.8 50.038 90)
 			(effects
@@
 			)
 		)
-		(property "Datasheet" "~"
+		(property "Datasheet" "https://hu.mouser.com/datasheet/2/348/esr_e-3009601.pdf"
 			(at 50.8 48.26 0)
 			(effects
@@
 			)
 		)
+		(property "Manufacturer_Part_Number" "ESR01MZPF20R0"
+			(at 50.8 48.26 0)
+			(effects
+				(font
+					(size 1.27 1.27)
+				)
+				(hide yes)
+			)
+		)
 		(pin "2"
 		)
@@
 			)
 		)
-		(property "Footprint" ""
+		(property "Footprint" "Diode_SMD:D_0603_1608Metric"
 			(at 63.5 69.85 0)
 			(effects
@@
 			)
 		)
-		(property "Datasheet" "~"
+		(property "Datasheet" "https://hu.mouser.com/datasheet/2/678/ASCKCx00_xxxxx0x0x02_DS101-3169121.pdf"
 			(at 63.5 69.85 0)
 			(effects
@@
 			)
 		)
+		(property "Manufacturer_Part_Number" "ASCKCA00-BU4V4020502"
+			(at 63.5 69.85 0)
+			(effects
+				(font
+					(size 1.27 1.27)
+				)
+				(hide yes)
+			)
+		)
 		(pin "1"
 		)
@@
 			)
 		)
-		(property "Footprint" ""
+		(property "Footprint" "Diode_SMD:D_0603_1608Metric"
 			(at 63.5 48.26 0)
 			(effects
@@
 			)
 		)
-		(property "Datasheet" "~"
+		(property "Datasheet" "https://hu.mouser.com/datasheet/2/678/ASCKCx00_xxxxx0x0x02_DS101-3169121.pdf"
 			(at 63.5 48.26 0)
 			(effects
@@
 			)
 		)
+		(property "Manufacturer_Part_Number" "ASCKCA00-BU4V4020502"
+			(at 63.5 48.26 0)
+			(effects
+				(font
+					(size 1.27 1.27)
+				)
+				(hide yes)
+			)
+		)
 		(pin "1"
 		)
@@
 			)
 		)
-		(property "Footprint" ""
+		(property "Footprint" "Diode_SMD:D_0603_1608Metric"
 			(at 63.5 81.28 0)
 			(effects
@@
 			)
 		)
-		(property "Datasheet" "~"
+		(property "Datasheet" "https://hu.mouser.com/datasheet/2/678/ASCKCx00_xxxxx0x0x02_DS101-3169121.pdf"
 			(at 63.5 81.28 0)
 			(effects
@@
 			(at 63.5 81.28 0)
 			(effects
+				(font
+					(size 1.27 1.27)
+				)
+				(hide yes)
+			)
+		)
+		(property "Manufacturer_Part_Number" "ASCKCA00-BU4V4020502"
+			(at 63.5 81.28 0)
+			(effects
