File: BMS/thermal.kicad_sch (KiCad schematic)
At the start: 6 parts

Commit message: DCDC fix unavailable parts, BMS redesign, handle fix, rearrange top half
Parts:
- C1: footprint (none) -> Capacitor_SMD:C_0805_2012Metric; Manufacturer_Part_Number (none) -> KGM21AR71H105JU
- R1: footprint (none) -> Resistor_SMD:R_0402_1005Metric; Manufacturer_Part_Number (none) -> CRCW040210K0FKEDC
- TH1, TH2, TH3, TH4: Manufacturer_Part_Number (none) -> 214650-1633
Changed lines of the file:
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@@
+			)
+		)
+		(property "Manufacturer_Part_Number" "214650-1633"
+			(at 67.31 62.23 0)
+			(effects
+				(font
+					(size 1.27 1.27)
+				)
+				(hide yes)
 			)
 		)
@@
 			)
 		)
+		(property "Manufacturer_Part_Number" "214650-1633"
+			(at 67.31 49.53 0)
+			(effects
+				(font
+					(size 1.27 1.27)
+				)
+				(hide yes)
+			)
+		)
 		(pin "1"
 		)
@@
 					(size 1.27 1.27)
 				)
+			)
+		)
+		(property "Manufacturer_Part_Number" "214650-1633"
+			(at 67.31 36.83 0)
+			(effects
+				(font
+					(size 1.27 1.27)
+				)
+				(hide yes)
 			)
 		)
@@
 			)
 		)
-		(property "Footprint" ""
+		(property "Footprint" "Resistor_SMD:R_0402_1005Metric"
 			(at 61.722 91.44 90)
 			(effects
@@
 			)
 		)
-		(property "Datasheet" "~"
+		(property "Datasheet" "https://www.vishay.com/docs/20035/dcrcwe3.pdf"
 			(at 63.5 91.44 0)
 			(effects
@@
 		)
 		(property "Description" "Resistor"
+			(at 63.5 91.44 0)
+			(effects
+				(font
+					(size 1.27 1.27)
+				)
+				(hide yes)
+			)
+		)
+		(property "Manufacturer_Part_Number" "CRCW040210K0FKEDC"
 			(at 63.5 91.44 0)
 			(effects
@@
 			)
 		)
-		(property "Footprint" ""
+		(property "Footprint" "Capacitor_SMD:C_0805_2012Metric"
 			(at 72.0852 104.14 0)
 			(effects
@@
 			)
 		)
-		(property "Datasheet" "~"
+		(property "Datasheet" "https://hu.mouser.com/datasheet/2/40/KGM_X7R-3223212.pdf"
 			(at 71.12 100.33 0)
 			(effects
@@
 		)
 		(property "Description" "Unpolarized capacitor"
+			(at 71.12 100.33 0)
+			(effects
+				(font
+					(size 1.27 1.27)
+				)
+				(hide yes)
+			)
+		)
+		(property "Manufacturer_Part_Number" "KGM21AR71H105JU"
 			(at 71.12 100.33 0)
 			(effects
@@
 			)
 		)
+		(property "Manufacturer_Part_Number" "214650-1633"
+			(at 67.31 76.2 0)
+			(effects
+				(font
+					(size 1.27 1.27)
+				)
+				(hide yes)
+			)
+		)
